Commit message: update readme

File: franka_description/robots/panda_arm_hand_simulation.urdf.xacro (robot description, xacro)
@@ -23,3 +23,24 @@
   <!-- Disable gravity of gripper -->
   <xacro:panda_gripper_gazebo />
+  <!-- add floor to avoid collision in moveit planning-->
+  <!-- <link name="wall">
+    <visual>
+      <geometry>
+        <box size="2 2 0.01"/>
+      </geometry>
+      <material name="gray"/>
+      <origin xyz="0 0 0.005" rpy="0 -0 0"/>
+    </visual>
+    <collision>
+      <geometry>
+        <box size="2 2 0.01"/>
+      </geometry>
+    </collision>
+    <xacro:default_inertial mass="1"/>
+  </link>
+  <joint name="world_wall_joint" type="fixed">
+    <parent link="world" />
+    <child link = "wall" />
+    <origin xyz="-0.0 0.0 -0.05" rpy="0.0 0.0 0.0" />
+  </joint> -->
 </robot>

Commit message: remove solutions

File: franka_description/robots/panda_arm_hand_simulation.urdf.xacro (robot description, xacro)
@@ -12,14 +12,10 @@
     </inertial>
   </xacro:macro>
-  <!-- incluude common stuff -->
+  <!-- include gazebo -->
   <xacro:include filename="$(find franka_description)/robots/panda.gazebo.xacro" />
-  <xacro:include filename="$(find franka_description)/robots/panda_arm.xacro"/>
-  <xacro:include filename="$(find franka_description)/robots/hand.xacro"/>
+  <!-- TODO: include xacro files for franka arm and hand -->
   <!-- TODO: create world link -->
-  <link name="world" />
   <!-- TODO: Franka arm -->
-  <xacro:panda_arm connected_to="world"/>
   <!-- TODO: Franka hand -->
-  <xacro:hand ns="panda" rpy="0 0 ${-pi/4}" connected_to="panda_link8"/>
   <!-- Disable gravity of gripper -->
   <xacro:panda_gripper_gazebo />
